File: hardware/schematic/schematic.kicad_pcb (KiCad board)
At the start: 2 copper layers, 65.5 x 45 mm, 25 parts, among them J1 Conn_01x09_Pin, J2 Conn_01x09_Pin, J3 ADS1115, J4 PE_SENSE_1, J7 PE_FORCE_IN, Q1 Q_NMOS_GSD, U1 LM317

Commit message: fixed schematic issue
Connections:
- J1 pad 5: /I2C_SDA -> /GP4
- J1 pad 7: /GP6 -> /I2C_SDA
Routing:
- net /I2C_SDA: track 37.9 -> 43.0 mm, vias 2 -> 3
Changed lines of the file:
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@@
 			(layers "*.Cu" "*.Mask")
 			(remove_unused_layers no)
-			(net "/I2C_SDA")
+			(net "/GP4")
 			(pinfunction "Pin_5_5")
-			(pintype "passive")
+			(pintype "passive+no_connect")
 		)
 		(pad "6" thru_hole circle
@@
 			(layers "*.Cu" "*.Mask")
 			(remove_unused_layers no)
-			(net "/GP6")
+			(net "/I2C_SDA")
 			(pinfunction "Pin_7_7")
-			(pintype "passive+no_connect")
+			(pintype "passive")
 		)
 		(pad "8" thru_hole circle
@@
 		(net "/I2C_SDA")
 	)
+	(segment
+		(start 120.5 111.08)
+		(end 125.12 106.46)
+		(width 0.2)
+		(layer "F.Cu")
+		(net "/I2C_SDA")
+	)
+	(segment
+		(start 120.5 116)
+		(end 120.5 111.08)
+		(width 0.2)
+		(layer "F.Cu")
+		(net "/I2C_SDA")
+	)
+	(via
+		(at 120.5 116)
+		(size 0.6)
+		(drill 0.3)
+		(layers "F.Cu" "B.Cu")
+		(net "/I2C_SDA")
+	)
 	(via
 		(at 115.725735 120.774265)
@@
 	)
 	(segment
-		(start 115.885735 120.774265)
-		(end 125.12 111.54)
-		(width 0.2)
-		(layer "B.Cu")
+		(start 115.725735 120.774265)
+		(end 120.5 116)
+		(width 0.2)
+		(layer "B.Cu")
