File: hardware/schematic/schematic.kicad_sch (KiCad schematic)
At the start: 0 parts

Commit message: schemativ v1.0
Parts:
- added C1: 100nF, Capacitor_THT:C_Disc_D5.0mm_W2.5mm_P2.50mm, symbol Device:C
- added D1: BAT54S, Package_TO_SOT_SMD:SOT-23, symbol Diode:BAT54S
- added J1, J2: Conn_01x09_Pin, Connector_PinHeader_2.54mm:PinHeader_1x09_P2.54mm_Vertical, symbol Connector:Conn_01x09_Pin
- added J3: ADS1115, Connector_PinHeader_2.54mm:PinHeader_1x09_P2.54mm_Vertical, symbol Connector:Conn_01x10_Pin
- added J4: PE_DUT, symbol Connector_Generic:Conn_01x02
- added J5: PE_DUT_RE, symbol Connector_Generic:Conn_01x02
- added R1: 6.2R / 1W, Resistor_THT:R_Axial_DIN0411_L9.9mm_D3.6mm_P12.70mm_Horizontal, symbol Device:R_US
- added R2: 10kR, Package_TO_SOT_SMD:SOT-23, symbol Device:R_US
- added U1: LM317, Package_TO_SOT_THT:TO-220-3_Vertical, symbol Regulator_Linear:LM317_TO-220
Connections:
- new net: R1.1, U1.2 (VO)
- new net: J4.2 (Pin_2), R1.2, U1.1 (ADJ)
- new net: J4.1 (Pin_1), R2.2
- new net 3V3: D1.2 (K), J2.7 (Pin_7), J3.10 (Pin_10)
- new net 5V: C1.1, J2.9 (Pin_9), U1.3 (VI)
- new net GND: J2.8 (Pin_8), J3.6 (Pin_6), J3.9 (Pin_9)
- new net GNDREF: C1.2, D1.1 (A), J5.2 (Pin_2)
- new net GP0: J1.1 (Pin_1)
- new net GP1: J1.2 (Pin_2)
- new net GP14: J2.1 (Pin_1)
- new net GP15: J2.2 (Pin_2)
- new net GP2: J1.3 (Pin_3)
- new net GP26: J2.3 (Pin_3)
- new net GP27: J2.4 (Pin_4)
- new net GP28: J2.5 (Pin_5)
- new net GP29: J2.6 (Pin_6)
- new net GP3: J1.4 (Pin_4)
- new net GP6: J1.7 (Pin_7)
- new net GP7: J1.8 (Pin_8)
- new net GP8: J1.9 (Pin_9)
- new net I2C_SCL: J1.5 (Pin_5), J3.8 (Pin_8)
- new net I2C_SDA: J1.6 (Pin_6), J3.7 (Pin_7)
- new net PE_TEST: D1.3 (COM), J3.4 (Pin_4), R2.1
- new net PE_TEST_RE: J3.3 (Pin_3), J5.1 (Pin_1)
- no-connect marks 0 -> 3

Commit message: finished schematic
Parts:
- removed J4: PE_DUT, symbol Connector_Generic:Conn_01x02
- removed J5: PE_DUT_RE, symbol Connector_Generic:Conn_01x02
- added D2, D3, D4: BAT54S, Package_TO_SOT_SMD:SOT-23, symbol Diode:BAT54S
- added J4: PE_SENSE_1, Connector_PinHeader_2.54mm:PinHeader_1x01_P2.54mm_Vertical, symbol Connector_Generic:Conn_01x01
- added J5: N_TEST, Connector_PinHeader_2.54mm:PinHeader_1x01_P2.54mm_Vertical, symbol Connector_Generic:Conn_01x01
- added J6: PE_SENSE_0, Connector_PinHeader_2.54mm:PinHeader_1x01_P2.54mm_Vertical, symbol Connector_Generic:Conn_01x01
- added J7: PE_FORCE_IN, Connector_PinHeader_2.54mm:PinHeader_1x01_P2.54mm_Vertical, symbol Connector_Generic:Conn_01x01
- added J8: PE_FORCE_OUT, Connector_PinHeader_2.54mm:PinHeader_1x01_P2.54mm_Vertical, symbol Connector_Generic:Conn_01x01
- added J9: L_TEST, Connector_PinHeader_2.54mm:PinHeader_1x01_P2.54mm_Vertical, symbol Connector_Generic:Conn_01x01
- added Q1: Q_NMOS_GSD, Package_TO_SOT_SMD:SOT-23, symbol Transistor_FET:Q_NMOS_GSD
- added R3, R4, R5: 10kR, Resistor_THT:R_Axial_DIN0207_L6.3mm_D2.5mm_P10.16mm_Horizontal, symbol Device:R_US
- added R6, R7: 1kR, Resistor_THT:R_Axial_DIN0207_L6.3mm_D2.5mm_P10.16mm_Horizontal, symbol Device:R_US
- J3: footprint Connector_PinHeader_2.54mm:PinHeader_1x09_P2.54mm_Vertical -> Connector_PinHeader_2.54mm:PinHeader_1x10_P2.54mm_Vertical
- R2: footprint Package_TO_SOT_SMD:SOT-23 -> Resistor_THT:R_Axial_DIN0207_L6.3mm_D2.5mm_P10.16mm_Horizontal
Connections:
- net 3V3: now also D2.2 (K), D3.2 (K), D4.2 (K)
- net GNDREF: now also D2.1 (A), D3.1 (A), D4.1 (A), J8.1 (Pin_1), Q1.2 (S)
- net GP26: now also R7.2
- net GP27: now also R6.1
- net I2C_SCL: now also J1.6 (Pin_6); no longer J1.5 (Pin_5)
- net I2C_SDA: now also J1.5 (Pin_5); no longer J1.6 (Pin_6)
- net PE_TEST_RE: now also D2.3 (COM), R3.2
- net at R1.2, U1.1 (ADJ): now also J7.1 (Pin_1)
- net at R2.2: now also J6.1 (Pin_1)
- net N_T: now reaches J3.1 (Pin_1)
- net N_T: now also D3.3 (COM), R4.1
- net L_T: now reaches J3.2 (Pin_2)
- net L_T: now also D4.3 (COM), R5.1
- net 5V: no longer names the net of C1.1, J2.9 (Pin_9), U1.3 (VI)
- new net: J9.1 (Pin_1), R5.2, R6.2
- new net: Q1.1 (G), R7.1
- new net: J5.1 (Pin_1), Q1.3 (D), R4.2
- new net: J4.1 (Pin_1), R3.1
- no-connect marks 3 -> 12
Other:
- moved on the sheet: D1, R2

Commit message: update
Parts:
- removed J5: N_TEST, Connector_PinHeader_2.54mm:PinHeader_1x01_P2.54mm_Vertical, symbol Connector_Generic:Conn_01x01
- removed J6: PE_SENSE_0, Connector_PinHeader_2.54mm:PinHeader_1x01_P2.54mm_Vertical, symbol Connector_Generic:Conn_01x01
- removed J8: PE_FORCE_OUT, Connector_PinHeader_2.54mm:PinHeader_1x01_P2.54mm_Vertical, symbol Connector_Generic:Conn_01x01
- removed J9: L_TEST, Connector_PinHeader_2.54mm:PinHeader_1x01_P2.54mm_Vertical, symbol Connector_Generic:Conn_01x01
- added L/N_TEST1, PE_OUT1: Conn_01x02, TerminalBlock_Phoenix:TerminalBlock_Phoenix_MKDS-1,5-2-5.08_1x02_P5.08mm_Horizontal, symbol Connector_Generic:Conn_01x02
Connections:
- net GND is gone; now on net GNDREF: J2.8 (Pin_8), J3.6 (Pin_6), J3.9 (Pin_9)
- net GNDREF: now also PE_OUT1.2 (Pin_2)
- net +5V: now reaches C1.1, J2.9 (Pin_9), U1.3 (VI)
- net at R5.2, R6.2: now also L/N_TEST1.1 (Pin_1)
- net N_TEST: now reaches Q1.3 (D), R4.2
- net N_TEST: now also L/N_TEST1.2 (Pin_2)
- net at R2.2: now also PE_OUT1.1 (Pin_1)
Other:
- moved on the sheet: D1, D4, R2, R5, R6

Commit message: fixed schematic issue
Connections:
- net GP6 is gone; now on net I2C_SDA: J1.7 (Pin_7)
- net I2C_SDA: no longer J1.5 (Pin_5)
- new net GP4: J1.5 (Pin_5)
Other:
- note added: "in reality gp2 (SDA), gp3(SCL) don't wonder"
Changed lines of the file:
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@@
 	(generator_version "10.0")
 	(paper "A4")
+	(text "in reality gp2 (SDA), gp3(SCL) don't wonder\n"
+		(exclude_from_sim no)
+		(at 117.094 133.604 0)
+		(effects
+			(font
+				(size 1.27 1.27)
+			)
+		)
+	)
 	(junction
 		(at 132.08 74.93)
@@
 	)
 	(no_connect
-		(at 121.92 121.92)
-	)
-	(no_connect
 		(at 101.6 124.46)
 	)
 	(no_connect
+		(at 121.92 124.46)
+	)
+	(no_connect
 		(at 121.92 111.76)
 	)
 	(no_connect
-		(at 121.92 124.46)
-	)
-	(no_connect
 		(at 213.36 113.03)
 	)
@@
 	)
 	(no_connect
+		(at 121.92 106.68)
+	)
+	(no_connect
 		(at 121.92 114.3)
 	)
 	(no_connect
-		(at 121.92 106.68)
+		(at 121.92 116.84)
 	)
 	(no_connect
@@
 		)
 	)
+	(label "N_TEST"
+		(at 135.89 74.93 0)
+		(effects
+			(font
+				(size 1.27 1.27)
+			)
+			(justify left bottom)
+		)
+	)
+	(label "3V3"
+		(at 133.35 96.52 90)
+		(effects
+			(font
+				(size 1.27 1.27)
+			)
+			(justify left bottom)
+		)
+	)
+	(label "I2C_SDA"
+		(at 121.92 121.92 0)
+		(effects
+			(font
+				(size 1.27 1.27)
+			)
+			(justify left bottom)
+		)
+	)
+	(label "3V3"
+		(at 187.96 86.36 0)
+		(effects
+			(font
+				(size 1.27 1.27)
+			)
+			(justify left bottom)
+		)
+	)
+	(label "PE_TEST"
+		(at 180.34 68.58 0)
+		(effects
+			(font
+				(size 1.27 1.27)
+			)
+			(justify left bottom)
+		)
+	)
+	(label "3V3"
+		(at 209.55 100.33 0)
+		(effects
+			(font
+				(size 1.27 1.27)
+			)
+			(justify left bottom)
+		)
+	)
+	(label "GP7"
+		(at 121.92 124.46 0)
+		(effects
+			(font
+				(size 1.27 1.27)
+			)
+			(justify left bottom)
+		)
+	)
+	(label "GP26"
+		(at 101.6 121.92 0)
+		(effects
+			(font
+				(size 1.27 1.27)
+			)
+			(justify left bottom)
+		)
+	)
+	(label "3V3"
+		(at 114.3 82.55 90)
+		(effects
+			(font
+				(size 1.27 1.27)
+			)
+			(justify left bottom)
+		)
+	)
+	(label "I2C_SCL"
+		(at 209.55 105.41 0)
+		(effects
+			(font
+				(size 1.27 1.27)
+			)
+			(justify left bottom)
+		)
+	)
+	(label "N_T"
+		(at 115.57 74.93 0)
+		(effects
+			(font
+				(size 1.27 1.27)
+			)
+			(justify left bottom)
+		)
+	)
+	(label "GP2"
+		(at 121.92 111.76 0)
+		(effects
+			(font
+				(size 1.27 1.27)
+			)
+			(justify left bottom)
+		)
+	)
+	(label "PE_TEST_RE"
+		(at 154.94 124.46 0)
+		(effects
+			(font
+				(size 1.27 1.27)
+			)
+			(justify left bottom)
+		)
+	)
 	(label "I2C_SCL"
 		(at 121.92 119.38 0)
@@
 	)
 	(label "N_TEST"
-		(at 135.89 74.93 0)
-		(effects
-			(font
-				(size 1.27 1.27)
-			)
-			(justify left bottom)
-		)
-	)
-	(label "3V3"
-		(at 133.35 96.52 90)
-		(effects
-			(font
-				(size 1.27 1.27)
-			)
-			(justify left bottom)
-		)
-	)
-	(label "GP6"
-		(at 121.92 121.92 0)
-		(effects
-			(font
-				(size 1.27 1.27)
-			)
-			(justify left bottom)
-		)
-	)
-	(label "3V3"
-		(at 187.96 86.36 0)
-		(effects
-			(font
-				(size 1.27 1.27)
-			)
-			(justify left bottom)
-		)
-	)
-	(label "PE_TEST"
-		(at 180.34 68.58 0)
-		(effects
-			(font
-				(size 1.27 1.27)
-			)
-			(justify left bottom)
-		)
-	)
-	(label "3V3"
-		(at 209.55 100.33 0)
-		(effects
-			(font
-				(size 1.27 1.27)
-			)
-			(justify left bottom)
-		)
-	)
-	(label "GP7"
-		(at 121.92 124.46 0)
-		(effects
-			(font
-				(size 1.27 1.27)
-			)
-			(justify left bottom)
-		)
-	)
-	(label "GP26"
-		(at 101.6 121.92 0)
-		(effects
-			(font
-				(size 1.27 1.27)
-			)
-			(justify left bottom)
-		)
-	)
-	(label "3V3"
-		(at 114.3 82.55 90)
-		(effects
-			(font
-				(size 1.27 1.27)
-			)
-			(justify left bottom)
-		)
-	)
-	(label "I2C_SCL"
-		(at 209.55 105.41 0)
-		(effects
-			(font
-				(size 1.27 1.27)
-			)
-			(justify left bottom)
-		)
-	)
-	(label "N_T"
-		(at 115.57 74.93 0)
-		(effects
-			(font
-				(size 1.27 1.27)
-			)
-			(justify left bottom)
-		)
-	)
-	(label "GP2"
-		(at 121.92 111.76 0)
-		(effects
-			(font
-				(size 1.27 1.27)
-			)
-			(justify left bottom)
-		)
-	)
-	(label "PE_TEST_RE"
-		(at 154.94 124.46 0)
-		(effects
-			(font
-				(size 1.27 1.27)
-			)
-			(justify left bottom)
-		)
-	)
-	(label "N_TEST"
 		(at 154.94 91.44 270)
 		(effects
@@
 		)
 	)
-	(label "I2C_SDA"
-		(at 121.92 116.84 0)
-		(effects
-			(font
-				(size 1.27 1.27)
-			)
-			(justify left bottom)
-		)
-	)
 	(label "GP3"
 		(at 121.92 114.3 0)
@@
 		(effects
 			(font
+				(size 1.27 1.27)
+			)
+			(justify left bottom)
+		)
+	)
+	(label "GP4"
+		(at 121.92 116.84 0)
+		(effects
+			(font

Commit message: added production files
Parts:
- D1, D2, D3, D4: LCSC (none) -> C83574
- Q1: LCSC (none) -> C20917
Changed lines of the file:
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@@
+			)
+		)
+		(property "LCSC" ""
+			(at 143.51 116.84 0)
+			(hide yes)
+			(show_name no)
+			(do_not_autoplace no)
+			(effects
+				(font
+					(size 1.27 1.27)
+				)
 			)
 		)
@@
 			)
 		)
+		(property "LCSC" "C83574"
+			(at 123.19 80.01 0)
+			(hide yes)
+			(show_name no)
+			(do_not_autoplace no)
+			(effects
+				(font
+					(size 1.27 1.27)
+				)
+			)
+		)
 		(pin "1"
 		)
@@
 			)
 		)
+		(property "LCSC" "C20917"
+			(at 134.62 63.5 0)
+			(hide yes)
+			(show_name no)
+			(do_not_autoplace no)
+			(effects
+				(font
+					(size 1.27 1.27)
+				)
+			)
+		)
 		(pin "2"
 		)
@@
 			)
 		)
+		(property "LCSC" ""
+			(at 160.02 88.9 0)
+			(hide yes)
+			(show_name no)
+			(do_not_autoplace no)
+			(effects
+				(font
+					(size 1.27 1.27)
+				)
+			)
+		)
 		(pin "1"
 		)
@@
 			)
 		)
+		(property "LCSC" ""
+			(at 143.51 63.5 90)
+			(hide yes)
+			(show_name no)
+			(do_not_autoplace no)
+			(effects
+				(font
+					(size 1.27 1.27)
+				)
+			)
+		)
 		(pin "2"
 		)
@@
 			)
 		)
+		(property "LCSC" ""
+			(at 168.91 110.49 90)
+			(hide yes)
+			(show_name no)
+			(do_not_autoplace no)
+			(effects
+				(font
+					(size 1.27 1.27)
+				)
+			)
+		)
 		(pin "1"
 		)
@@
 			)
 		)
+		(property "LCSC" ""
+			(at 116.84 116.84 0)
+			(hide yes)
+			(show_name no)
+			(do_not_autoplace no)
+			(effects
+				(font
+					(size 1.27 1.27)
+				)
+			)
+		)
 		(pin "4"
 		)
@@
 		)
 		(property "Description" "Resistor, US symbol"
+			(at 151.13 81.28 0)
+			(hide yes)
+			(show_name no)
+			(do_not_autoplace no)
+			(effects
+				(font
+					(size 1.27 1.27)
+				)
+			)
+		)
+		(property "LCSC" ""
 			(at 151.13 81.28 0)
 			(hide yes)
@@
 			)
 		)
+		(property "LCSC" ""
+			(at 184.15 110.49 0)
+			(hide yes)
+			(show_name no)
+			(do_not_autoplace no)
+			(effects
+				(font
+					(size 1.27 1.27)
+				)
+			)
+		)
 		(pin "1"
 		)
@@
 			)
 		)
+		(property "LCSC" ""
+			(at 185.42 95.25 0)
+			(hide yes)
+			(show_name no)
+			(do_not_autoplace no)
+			(effects
+				(font
+					(size 1.27 1.27)
+				)
+			)
+		)
 		(pin "2"
 		)
@@
 			)
 		)
+		(property "LCSC" ""
+			(at 106.68 116.84 0)
+			(hide yes)
+			(show_name no)
+			(do_not_autoplace no)
+			(effects
+				(font
+					(size 1.27 1.27)
+				)
+			)
+		)
 		(pin "6"
 		)
@@
 			)
 		)
+		(property "LCSC" ""
+			(at 184.15 124.46 0)
+			(hide yes)
+			(show_name no)
+			(do_not_autoplace no)
+			(effects
+				(font
+					(size 1.27 1.27)
+				)
+			)
+		)
 		(pin "1"
 		)
@@
 		(property "Description" "Resistor, US symbol"
 			(at 171.45 124.46 0)
+			(hide yes)
+			(show_name no)
+			(do_not_autoplace no)
+			(effects
+				(font
+					(size 1.27 1.27)
+				)
+			)
+		)
+		(property "LCSC" ""
+			(at 171.45 124.46 90)
 			(hide yes)
 			(show_name no)
@@
 			)
 		)
+		(property "LCSC" "C83574"
+			(at 142.24 93.98 0)
+			(hide yes)
+			(show_name no)
+			(do_not_autoplace no)
+			(effects
+				(font
+					(size 1.27 1.27)
+				)
+			)
+		)
 		(pin "1"
 		)
@@
 			)
 		)
+		(property "LCSC" "C83574"
+			(at 162.56 129.54 0)
+			(hide yes)
+			(show_name no)
+			(do_not_autoplace no)
+			(effects
+				(font
+					(size 1.27 1.27)
+				)
+			)
+		)
 		(pin "3"
 		)
@@
 			)
 		)
+		(property "LCSC" "C83574"
+			(at 185.42 78.74 90)
+			(hide yes)
+			(show_name no)
+			(do_not_autoplace no)
+			(effects
+				(font
+					(size 1.27 1.27)
+				)
+			)
+		)
 		(pin "2"
 		)
@@
 		)
 		(property "Description" "Generic connector, single row, 01x10, script generated"
+			(at 218.44 113.03 0)
+			(hide yes)
+			(show_name no)
+			(do_not_autoplace no)
+			(effects
+				(font
+					(size 1.27 1.27)
+				)
+			)
+		)
+		(property "LCSC" ""
 			(at 218.44 113.03 0)
 			(hide yes)
@@
 			)
 		)
+		(property "LCSC" ""
+			(at 128.27 74.93 90)
+			(hide yes)
+			(show_name no)
+			(do_not_autoplace no)
+			(effects
+				(font
+					(size 1.27 1.27)
+				)
+			)
+		)
 		(pin "2"
 		)
@@
 			)
 		)
+		(property "LCSC" ""
+			(at 154.94 110.49 0)
+			(hide yes)
+			(show_name no)
+			(do_not_autoplace no)
+			(effects
+				(font
+					(size 1.27 1.27)
+				)
+			)
+		)
 		(pin "1"
 		)
@@
 			)
 		)
+		(property "LCSC" ""
+			(at 180.34 90.17 0)
+			(hide yes)
+			(show_name no)
+			(do_not_autoplace no)
+			(effects
+				(font
+					(size 1.27 1.27)
+				)
+			)
+		)
 		(pin "2"
 		)
@@
 			(hide yes)
 			(show_name no)
+			(do_not_autoplace no)
+			(effects
+				(font
+					(size 1.27 1.27)
+				)
+			)
+		)
+		(property "LCSC" ""
+			(at 147.32 88.9 90)
+			(hide yes)
+			(show_name no)
